Commit message: Fix LiDAR sensor type and bridge topic paths
- lidar_ign.xacro: revert to gpu_lidar/lidar (the correct Ignition-native
  type). type=ray is Gazebo Classic only — Ignition never registers it or
  publishes to any topic. Remove <frame_id> which breaks SDF conversion.
- gz_bridge.yaml: fix IMU gz_topic_name to the actual scoped Ignition topic
  path confirmed by ign topic -l output.
- industrial.sdf: user change to libignition-gazebo-sensors-system.so filename.

Co-Authored-By: Claude Sonnet 4.6 <noreply@anthropic.com>

File: src/go2_ign_bringup/xacro/lidar_ign.xacro (robot description, xacro)
@@ -21,5 +21,5 @@
       <origin rpy="0 0 0" xyz="0 0 0"/>
       <geometry>
-        <mesh filename="file://$(find go2_description)/meshes/hokuyo.dae"/>
+        <box size="0.07 0.07 0.07"/>
       </geometry>
     </visual>
@@ -31,17 +31,20 @@
   </link>
   <!--
-    type="ray" is the Ignition Gazebo Fortress CPU-based lidar sensor.
-    It publishes ignition.msgs.LaserScan to the topic set below.
-    - Do NOT use <frame_id>: it is not valid SDF and breaks sensor conversion.
-    - Do NOT use type="gpu_lidar": requires a GPU render context that may not
-      be available inside the container and uses <lidar> not <ray>.
-    - The absolute topic /scan is bridged to ROS by gz_bridge.yaml.
+    gpu_lidar is the correct Ignition Gazebo Fortress native sensor type for lidar.
+    type="ray" is a Gazebo Classic type — Ignition does not publish it to any topic.
+    Rules:
+      - Use <lidar> (NOT <ray>) as the inner element for gpu_lidar.
+      - Do NOT add <frame_id>: it is not valid SDF and silently kills the sensor
+        during URDF-to-SDF conversion (the sensor disappears from the model).
+      - <topic>/scan</topic> sets an absolute Ignition topic path (leading / = absolute).
+        The Sensors world plugin bridges it; ros_ign_bridge maps it to ROS /scan.
   -->
   <gazebo reference="front_laser">
-    <sensor name="front_laser_sensor" type="ray">
+    <sensor name="front_laser_sensor" type="gpu_lidar">
       <always_on>true</always_on>
       <visualize>true</visualize>
       <update_rate>10</update_rate>
-      <ray>
+      <topic>/scan</topic>
+      <lidar>
         <scan>
           <horizontal>
@@ -62,6 +65,5 @@
           <stddev>0.01</stddev>
         </noise>
-      </ray>
-      <topic>/scan</topic>
+      </lidar>
     </sensor>
   </gazebo>
